File: Giger-counter-addon.kicad_sch (KiCad schematic)
At the start: 22 parts, among them J1 Expanction, J2 Beeper, J3 Giger counter conn, J4 FTDI, J5 power-in, J6 Barrel_Jack_Switch, U1 LM2596S-5, U2 LM1117-3.3, U3 ESP8266-12F

Commit message: cleaned up some notes
Other:
- note added: "Ignore or disconnect GPIO 0 and Reset for ftdi connenter."
- note added: "giger counter refrance https://circuitmaker.com/Projects/Details/YannickVerbelen/Geiger-Counter"
- note added: "optonal expantion"
- note removed: "barrel jack form labitat power input use MCH lighs for footprint"
- note removed: "https://circuitmaker.com/Projects/Details/YannickVerbelen/Geiger-Counter"
Changed lines of the file:
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@@
     (stroke (width 0) (type default) (color 0 0 0 0))
+  )
+  (text "Ignore or disconnect GPIO 0 and Reset for ftdi connenter.\n"
+    (at 198.12 140.335 0)
+    (effects (font (size 1.27 1.27)) (justify left bottom))
+  )
+  (text "optonal expantion 	" (at 118.11 36.83 0)
+    (effects (font (size 1.27 1.27)) (justify left bottom))
   )
   (text "NR6045T680M - inductor\nNSR0530HT1G - revser diode" (at 73.66 127 0)
     (effects (font (size 1.27 1.27)) (justify left bottom))
   )
-  (text "https://circuitmaker.com/Projects/Details/YannickVerbelen/Geiger-Counter"
+  (text "giger counter refrance\nhttps://circuitmaker.com/Projects/Details/YannickVerbelen/Geiger-Counter"
     (at 50.8 147.32 0)
     (effects (font (size 1.27 1.27)) (justify left bottom))
   )
-  (text "barrel jack form labitat power input\nuse MCH lighs for footprint\n"
-    (at 45.72 48.26 0)
-    (effects (font (size 1.27 1.27)) (justify left bottom))
-  )
